Commit message: feat: update simulation launch files and enhance README documentation
- Replaced `headless_sim.launch.py` with `simulate.launch.py` for improved simulation management.
- Introduced new launch files: `test.launch.py` for debugging and `fake_pub.launch.py` for demonstration purposes.
- Updated README files to reflect changes in launch commands and provide clearer instructions on simulation and SLAM integration.
- Enhanced `.gitignore` to exclude additional cache directories.
- Refactored `ros_tf_bridge.py` and `server.py` to align with new launch configurations.

File: src/simulate/simulate/urdf/simple_2d_robot.urdf.xacro (robot description, xacro)
@@ -1,4 +1,15 @@
 <?xml version="1.0"?>
 <robot name="simple_2d_robot" xmlns:xacro="http://www.ros.org/wiki/xacro">
+  <!-- robot_namespace: ROS node namespace for Gazebo plugins. frame_prefix: TF link prefix, e.g. "robot2/" or "" for global. -->
+  <xacro:arg name="robot_namespace" default="/"/>
+  <xacro:arg name="frame_prefix" default=""/>
+  <xacro:property name="lnk_bf" value="$(arg frame_prefix)base_footprint"/>
+  <xacro:property name="lnk_base" value="$(arg frame_prefix)base_link"/>
+  <xacro:property name="lnk_lw" value="$(arg frame_prefix)left_wheel_link"/>
+  <xacro:property name="lnk_rw" value="$(arg frame_prefix)right_wheel_link"/>
+  <xacro:property name="lnk_laser" value="$(arg frame_prefix)laser_link"/>
+  <xacro:property name="lnk_imu" value="$(arg frame_prefix)imu_link"/>
+  <xacro:property name="lnk_cam" value="$(arg frame_prefix)camera_link"/>
+  <xacro:property name="lnk_odom" value="$(arg frame_prefix)odom"/>
   <xacro:property name="base_length" value="0.40"/>
   <xacro:property name="base_width" value="0.30"/>
@@ -7,12 +18,11 @@
   <xacro:property name="wheel_width" value="0.03"/>
   <xacro:property name="wheel_sep" value="0.26"/>
-  <!-- Massless root: KDL-friendly; odom TF attaches here (see diff_drive robot_base_frame). -->
-  <link name="base_footprint"/>
+  <link name="${lnk_bf}"/>
   <joint name="base_footprint_joint" type="fixed">
-    <parent link="base_footprint"/>
-    <child link="base_link"/>
+    <parent link="${lnk_bf}"/>
+    <child link="${lnk_base}"/>
     <origin xyz="0 0 0" rpy="0 0 0"/>
   </joint>
-  <link name="base_link">
+  <link name="${lnk_base}">
     <inertial>
       <origin xyz="0 0 0"/>
@@ -36,5 +46,5 @@
     </collision>
   </link>
-  <link name="left_wheel_link">
+  <link name="${lnk_lw}">
     <inertial>
       <origin xyz="0 0 0"/>
@@ -58,5 +68,5 @@
     </collision>
   </link>
-  <link name="right_wheel_link">
+  <link name="${lnk_rw}">
     <inertial>
       <origin xyz="0 0 0"/>
@@ -79,16 +89,16 @@
   </link>
   <joint name="left_wheel_joint" type="continuous">
-    <parent link="base_link"/>
-    <child link="left_wheel_link"/>
+    <parent link="${lnk_base}"/>
+    <child link="${lnk_lw}"/>
     <origin xyz="0 ${wheel_sep/2} ${wheel_radius}" rpy="0 0 0"/>
     <axis xyz="0 1 0"/>
   </joint>
   <joint name="right_wheel_joint" type="continuous">
-    <parent link="base_link"/>
-    <child link="right_wheel_link"/>
+    <parent link="${lnk_base}"/>
+    <child link="${lnk_rw}"/>
     <origin xyz="0 ${-wheel_sep/2} ${wheel_radius}" rpy="0 0 0"/>
     <axis xyz="0 1 0"/>
   </joint>
-  <link name="laser_link">
+  <link name="${lnk_laser}">
     <inertial>
       <origin xyz="0 0 0"/>
@@ -106,9 +116,9 @@
   </link>
   <joint name="laser_joint" type="fixed">
-    <parent link="base_link"/>
-    <child link="laser_link"/>
+    <parent link="${lnk_base}"/>
+    <child link="${lnk_laser}"/>
     <origin xyz="0.12 0 ${base_height + 0.03}" rpy="0 0 0"/>
   </joint>
-  <link name="imu_link">
+  <link name="${lnk_imu}">
     <inertial>
       <origin xyz="0 0 0"/>
@@ -118,9 +128,9 @@
   </link>
   <joint name="imu_joint" type="fixed">
-    <parent link="base_link"/>
-    <child link="imu_link"/>
+    <parent link="${lnk_base}"/>
+    <child link="${lnk_imu}"/>
     <origin xyz="0 0 ${base_height + 0.02}" rpy="0 0 0"/>
   </joint>
-  <link name="camera_link">
+  <link name="${lnk_cam}">
     <inertial>
       <origin xyz="0 0 0"/>
@@ -138,17 +148,17 @@
   </link>
   <joint name="camera_joint" type="fixed">
-    <parent link="base_link"/>
-    <child link="camera_link"/>
+    <parent link="${lnk_base}"/>
+    <child link="${lnk_cam}"/>
     <origin xyz="0.18 0 ${base_height + 0.05}" rpy="0 0 0"/>
   </joint>
-  <gazebo reference="left_wheel_link">
+  <gazebo reference="${lnk_lw}">
     <mu1>2.0</mu1>
     <mu2>2.0</mu2>
   </gazebo>
-  <gazebo reference="right_wheel_link">
+  <gazebo reference="${lnk_rw}">
     <mu1>2.0</mu1>
     <mu2>2.0</mu2>
   </gazebo>
-  <gazebo reference="laser_link">
+  <gazebo reference="${lnk_laser}">
     <sensor type="ray" name="scan">
       <always_on>true</always_on>
@@ -172,13 +182,13 @@
       <plugin name="laser_controller" filename="libgazebo_ros_ray_sensor.so">
         <ros>
-          <namespace>/</namespace>
+          <namespace>$(arg robot_namespace)</namespace>
           <remapping>~/out:=scan</remapping>
         </ros>
         <output_type>sensor_msgs/LaserScan</output_type>
-        <frame_name>laser_link</frame_name>
+        <frame_name>${lnk_laser}</frame_name>
       </plugin>
     </sensor>
   </gazebo>
-  <gazebo reference="imu_link">
+  <gazebo reference="${lnk_imu}">
     <sensor type="imu" name="imu_sensor">
       <always_on>true</always_on>
@@ -186,12 +196,12 @@
       <plugin name="imu_plugin" filename="libgazebo_ros_imu_sensor.so">
         <ros>
-          <namespace>/</namespace>
+          <namespace>$(arg robot_namespace)</namespace>
           <remapping>~/out:=imu/data</remapping>
         </ros>
-        <frame_name>imu_link</frame_name>
+        <frame_name>${lnk_imu}</frame_name>
       </plugin>
     </sensor>
   </gazebo>
-  <gazebo reference="camera_link">
+  <gazebo reference="${lnk_cam}">
     <sensor type="camera" name="front_camera">
       <always_on>true</always_on>
@@ -211,9 +221,9 @@
       <plugin name="camera_controller" filename="libgazebo_ros_camera.so">
         <ros>
-          <namespace>/</namespace>
+          <namespace>$(arg robot_namespace)</namespace>
           <remapping>~/image_raw:=camera/image_raw</remapping>
           <remapping>~/camera_info:=camera/camera_info</remapping>
         </ros>
-        <frame_name>camera_link</frame_name>
+        <frame_name>${lnk_cam}</frame_name>
       </plugin>
     </sensor>
@@ -222,5 +232,5 @@
     <plugin name="diff_drive_controller" filename="libgazebo_ros_diff_drive.so">
       <ros>
-        <namespace>/</namespace>
+        <namespace>$(arg robot_namespace)</namespace>
       </ros>
       <update_rate>50</update_rate>
@@ -233,6 +243,6 @@
       <command_topic>cmd_vel</command_topic>
       <odometry_topic>odom</odometry_topic>
-      <odometry_frame>odom</odometry_frame>
-      <robot_base_frame>base_footprint</robot_base_frame>
+      <odometry_frame>${lnk_odom}</odometry_frame>
+      <robot_base_frame>${lnk_bf}</robot_base_frame>
       <publish_odom>true</publish_odom>
       <publish_odom_tf>true</publish_odom_tf>
