Commit message: feat: improve multi-robot simulation sensing

File: src/simulate/simulate/urdf/simple_2d_robot.urdf.xacro (robot description, xacro)
@@ -4,4 +4,6 @@
   <xacro:arg name="robot_namespace" default="/"/>
   <xacro:arg name="frame_prefix" default=""/>
+  <xacro:arg name="collision_bit" default="4"/>
+  <xacro:arg name="collision_filter_plugin" default="libray_collision_filter_plugin.so"/>
   <xacro:property name="lnk_bf" value="$(arg frame_prefix)base_footprint"/>
   <xacro:property name="lnk_base" value="$(arg frame_prefix)base_link"/>
@@ -11,8 +13,13 @@
   <xacro:property name="lnk_imu" value="$(arg frame_prefix)imu_link"/>
   <xacro:property name="lnk_cam" value="$(arg frame_prefix)camera_link"/>
+  <xacro:property name="lnk_down_cam" value="$(arg frame_prefix)front_down_camera_link"/>
   <xacro:property name="lnk_odom" value="$(arg frame_prefix)odom"/>
   <xacro:property name="base_length" value="0.40"/>
   <xacro:property name="base_width" value="0.30"/>
   <xacro:property name="base_height" value="0.12"/>
+  <!-- The lidar plane crosses this shell, so other robots see the complete body outline. -->
+  <xacro:property name="shell_length" value="0.42"/>
+  <xacro:property name="shell_width" value="0.32"/>
+  <xacro:property name="shell_height" value="0.22"/>
   <xacro:property name="wheel_radius" value="0.06"/>
   <xacro:property name="wheel_width" value="0.03"/>
@@ -46,4 +53,21 @@
     </collision>
   </link>
+  <!-- Full-height collision shell makes the robot visible in peer lidar scans. -->
+  <link name="$(arg frame_prefix)outer_shell_link">
+    <visual>
+      <origin xyz="0 0 ${shell_height/2}"/>
+      <geometry><box size="${shell_length} ${shell_width} ${shell_height}"/></geometry>
+      <material name="shell_gray"><color rgba="0.42 0.45 0.50 1.0"/></material>
+    </visual>
+    <collision>
+      <origin xyz="0 0 ${shell_height/2}"/>
+      <geometry><box size="${shell_length} ${shell_width} ${shell_height}"/></geometry>
+    </collision>
+  </link>
+  <joint name="outer_shell_joint" type="fixed">
+    <parent link="${lnk_base}"/>
+    <child link="$(arg frame_prefix)outer_shell_link"/>
+    <origin xyz="0 0 0" rpy="0 0 0"/>
+  </joint>
   <link name="${lnk_lw}">
     <inertial>
@@ -118,5 +142,5 @@
     <parent link="${lnk_base}"/>
     <child link="${lnk_laser}"/>
-    <origin xyz="0.12 0 ${base_height + 0.03}" rpy="0 0 0"/>
+    <origin xyz="0.23 0 ${base_height + 0.03}" rpy="0 0 0"/>
   </joint>
   <link name="${lnk_imu}">
@@ -151,4 +175,21 @@
     <child link="${lnk_cam}"/>
     <origin xyz="0.18 0 ${base_height + 0.05}" rpy="0 0 0"/>
+  </joint>
+  <link name="${lnk_down_cam}">
+    <inertial>
+      <origin xyz="0 0 0"/>
+      <mass value="0.15"/>
+      <inertia ixx="0.0002" ixy="0.0" ixz="0.0" iyy="0.0002" iyz="0.0" izz="0.0002"/>
+    </inertial>
+    <visual>
+      <geometry><box size="0.05 0.05 0.04"/></geometry>
+      <material name="down_camera_green"><color rgba="0.05 0.55 0.18 1.0"/></material>
+    </visual>
+  </link>
+  <joint name="front_down_camera_joint" type="fixed">
+    <parent link="${lnk_base}"/>
+    <child link="${lnk_down_cam}"/>
+    <!-- Positive pitch rotates the camera +X optical axis toward the floor. -->
+    <origin xyz="0.19 0 0.18" rpy="0 0.436332 0"/>
   </joint>
   <gazebo reference="${lnk_lw}">
@@ -170,6 +211,6 @@
             <samples>720</samples>
             <resolution>1</resolution>
-            <min_angle>-3.14159</min_angle>
-            <max_angle>3.14159</max_angle>
+            <min_angle>-1.5708</min_angle>
+            <max_angle>1.5708</max_angle>
           </horizontal>
         </scan>
@@ -180,4 +221,8 @@
         </range>
       </ray>
+      <plugin name="ray_collision_filter" filename="$(arg collision_filter_plugin)">
+        <own_category_bits>$(arg collision_bit)</own_category_bits>
+        <shell_link>$(arg frame_prefix)outer_shell_link</shell_link>
+      </plugin>
       <plugin name="laser_controller" filename="libgazebo_ros_ray_sensor.so">
         <ros>
@@ -229,4 +274,24 @@
     </sensor>
   </gazebo>
+  <gazebo reference="${lnk_down_cam}">
+    <sensor type="camera" name="front_down_camera">
+      <always_on>true</always_on>
+      <visualize>false</visualize>
+      <update_rate>15</update_rate>
+      <camera name="front_down_camera">
+        <horizontal_fov>1.047</horizontal_fov>
+        <image><width>640</width><height>480</height><format>R8G8B8</format></image>
+        <clip><near>0.05</near><far>15</far></clip>
+      </camera>
+      <plugin name="front_down_camera_controller" filename="libgazebo_ros_camera.so">
+        <ros>
+          <namespace>$(arg robot_namespace)</namespace>
+          <remapping>~/image_raw:=front_down_camera/image_raw</remapping>
+          <remapping>~/camera_info:=front_down_camera/camera_info</remapping>
+        </ros>
+        <frame_name>${lnk_down_cam}</frame_name>
+      </plugin>
+    </sensor>
+  </gazebo>
   <gazebo>
     <plugin name="diff_drive_controller" filename="libgazebo_ros_diff_drive.so">

Commit message: fix(gazebo): complete topdown camera controls

File: src/simulate/simulate/urdf/simple_2d_robot.urdf.xacro (robot description, xacro)
@@ -190,6 +190,7 @@
     <parent link="${lnk_base}"/>
     <child link="${lnk_down_cam}"/>
+    <!-- Keep the lens ahead of the 0.42 m shell so the body is outside the image. -->
     <!-- Positive pitch rotates the camera +X optical axis toward the floor. -->
-    <origin xyz="0.19 0 0.18" rpy="0 0.436332 0"/>
+    <origin xyz="0.28 0 0.18" rpy="0 0.436332 0"/>
   </joint>
   <gazebo reference="${lnk_lw}">

Commit message: Improve bag replay and web monitoring

File: src/simulate/simulate/urdf/simple_2d_robot.urdf.xacro (robot description, xacro)
@@ -174,5 +174,6 @@
     <parent link="${lnk_base}"/>
     <child link="${lnk_cam}"/>
-    <origin xyz="0.18 0 ${base_height + 0.05}" rpy="0 0 0"/>
+    <!-- Keep the camera body and optical origin ahead of the outer shell. -->
+    <origin xyz="${shell_length/2 + 0.03} 0 ${base_height + 0.05}" rpy="0 0 0"/>
   </joint>
   <link name="${lnk_down_cam}">

Commit message: feat: add per-robot navigation settings and improve simulation web controls

File: src/simulate/simulate/urdf/simple_2d_robot.urdf.xacro (robot description, xacro)
@@ -14,4 +14,6 @@
   <xacro:property name="lnk_cam" value="$(arg frame_prefix)camera_link"/>
   <xacro:property name="lnk_down_cam" value="$(arg frame_prefix)front_down_camera_link"/>
+  <xacro:property name="lnk_top_marker" value="$(arg frame_prefix)top_marker_link"/>
+  <xacro:property name="lnk_heading_marker" value="$(arg frame_prefix)heading_marker_link"/>
   <xacro:property name="lnk_odom" value="$(arg frame_prefix)odom"/>
   <xacro:property name="base_length" value="0.40"/>
@@ -70,4 +72,35 @@
     <origin xyz="0 0 0" rpy="0 0 0"/>
   </joint>
+  <!-- High-visibility roof plate for the 32 m overhead Gazebo camera. It has
+       no collision geometry, so navigation, lidar and body footprint stay unchanged. -->
+  <link name="${lnk_top_marker}">
+    <visual>
+      <origin xyz="0 0 0"/>
+      <geometry><box size="0.38 0.27 0.012"/></geometry>
+      <material name="high_visibility_orange">
+        <color rgba="1.0 0.28 0.0 1.0"/>
+      </material>
+    </visual>
+  </link>
+  <joint name="top_marker_joint" type="fixed">
+    <parent link="${lnk_base}"/>
+    <child link="${lnk_top_marker}"/>
+    <origin xyz="0 0 ${shell_height + 0.008}" rpy="0 0 0"/>
+  </joint>
+  <!-- Contrasting front stripe makes robot heading legible from directly above. -->
+  <link name="${lnk_heading_marker}">
+    <visual>
+      <origin xyz="0 0 0"/>
+      <geometry><box size="0.09 0.23 0.008"/></geometry>
+      <material name="heading_white">
+        <color rgba="1.0 1.0 1.0 1.0"/>
+      </material>
+    </visual>
+  </link>
+  <joint name="heading_marker_joint" type="fixed">
+    <parent link="${lnk_base}"/>
+    <child link="${lnk_heading_marker}"/>
+    <origin xyz="0.135 0 ${shell_height + 0.020}" rpy="0 0 0"/>
+  </joint>
   <link name="${lnk_lw}">
     <inertial>
@@ -202,4 +235,10 @@
     <mu1>2.0</mu1>
     <mu2>2.0</mu2>
+  </gazebo>
+  <gazebo reference="${lnk_top_marker}">
+    <material>Gazebo/Orange</material>
+  </gazebo>
+  <gazebo reference="${lnk_heading_marker}">
+    <material>Gazebo/White</material>
   </gazebo>
   <gazebo reference="${lnk_laser}">

Commit message: Validate simulated robot model and refine sensor geometry

File: src/simulate/simulate/urdf/simple_2d_robot.urdf.xacro (robot description, xacro)
@@ -17,11 +17,14 @@
   <xacro:property name="lnk_heading_marker" value="$(arg frame_prefix)heading_marker_link"/>
   <xacro:property name="lnk_odom" value="$(arg frame_prefix)odom"/>
-  <xacro:property name="base_length" value="0.40"/>
-  <xacro:property name="base_width" value="0.30"/>
-  <xacro:property name="base_height" value="0.12"/>
+  <xacro:property name="base_length" value="0.38"/>
+  <xacro:property name="base_width" value="0.22"/>
+  <xacro:property name="base_height" value="0.08"/>
+  <xacro:property name="ground_clearance" value="0.035"/>
+  <xacro:property name="shell_bottom" value="0.125"/>
+  <xacro:property name="roof_height" value="0.24"/>
   <!-- The lidar plane crosses this shell, so other robots see the complete body outline. -->
   <xacro:property name="shell_length" value="0.42"/>
   <xacro:property name="shell_width" value="0.32"/>
-  <xacro:property name="shell_height" value="0.22"/>
+  <xacro:property name="shell_height" value="0.115"/>
   <xacro:property name="wheel_radius" value="0.06"/>
   <xacro:property name="wheel_width" value="0.03"/>
@@ -35,10 +38,10 @@
   <link name="${lnk_base}">
     <inertial>
-      <origin xyz="0 0 0"/>
+      <origin xyz="0 0 0.09"/>
       <mass value="12.0"/>
-      <inertia ixx="0.12" ixy="0.0" ixz="0.0" iyy="0.12" iyz="0.0" izz="0.20"/>
-    </inertial>
-    <visual>
-      <origin xyz="0 0 ${base_height/2}"/>
+      <inertia ixx="0.12" ixy="0.0" ixz="0.0" iyy="0.20" iyz="0.0" izz="0.25"/>
+    </inertial>
+    <visual>
+      <origin xyz="0 0 ${ground_clearance + base_height/2}"/>
       <geometry>
         <box size="${base_length} ${base_width} ${base_height}"/>
@@ -49,5 +52,5 @@
     </visual>
     <collision>
-      <origin xyz="0 0 ${base_height/2}"/>
+      <origin xyz="0 0 ${ground_clearance + base_height/2}"/>
       <geometry>
         <box size="${base_length} ${base_width} ${base_height}"/>
@@ -58,10 +61,10 @@
   <link name="$(arg frame_prefix)outer_shell_link">
     <visual>
-      <origin xyz="0 0 ${shell_height/2}"/>
+      <origin xyz="0 0 ${shell_bottom + shell_height/2}"/>
       <geometry><box size="${shell_length} ${shell_width} ${shell_height}"/></geometry>
-      <material name="shell_gray"><color rgba="0.42 0.45 0.50 1.0"/></material>
+      <material name="shell_gray"><color rgba="0.84 0.88 0.92 1.0"/></material>
     </visual>
     <collision>
-      <origin xyz="0 0 ${shell_height/2}"/>
+      <origin xyz="0 0 ${shell_bottom + shell_height/2}"/>
       <geometry><box size="${shell_length} ${shell_width} ${shell_height}"/></geometry>
     </collision>
@@ -86,5 +89,5 @@
     <parent link="${lnk_base}"/>
     <child link="${lnk_top_marker}"/>
-    <origin xyz="0 0 ${shell_height + 0.008}" rpy="0 0 0"/>
+    <origin xyz="0 0 ${roof_height + 0.008}" rpy="0 0 0"/>
   </joint>
   <!-- Contrasting front stripe makes robot heading legible from directly above. -->
@@ -101,5 +104,5 @@
     <parent link="${lnk_base}"/>
     <child link="${lnk_heading_marker}"/>
-    <origin xyz="0.135 0 ${shell_height + 0.020}" rpy="0 0 0"/>
+    <origin xyz="0.135 0 ${roof_height + 0.020}" rpy="0 0 0"/>
   </joint>
   <link name="${lnk_lw}">
@@ -171,9 +174,13 @@
       </material>
     </visual>
+  <collision>
+      <origin xyz="0 0 0"/>
+      <geometry><cylinder radius="0.03" length="0.04"/></geometry>
+    </collision>
   </link>
   <joint name="laser_joint" type="fixed">
     <parent link="${lnk_base}"/>
     <child link="${lnk_laser}"/>
-    <origin xyz="0.23 0 ${base_height + 0.03}" rpy="0 0 0"/>
+    <origin xyz="0.23 0 0.17" rpy="0 0 0"/>
   </joint>
   <link name="${lnk_imu}">
@@ -187,5 +194,5 @@
     <parent link="${lnk_base}"/>
     <child link="${lnk_imu}"/>
-    <origin xyz="0 0 ${base_height + 0.02}" rpy="0 0 0"/>
+    <origin xyz="0 0 0.12" rpy="0 0 0"/>
   </joint>
   <link name="${lnk_cam}">
@@ -196,11 +203,16 @@
     </inertial>
     <visual>
+      <origin xyz="-0.022 0 0"/>
       <geometry>
         <box size="0.04 0.04 0.03"/>
       </geometry>
       <material name="green">
-        <color rgba="0.1 0.7 0.2 1.0"/>
-      </material>
-    </visual>
+        <color rgba="0.04 0.06 0.09 1.0"/>
+      </material>
+    </visual>
+  <collision>
+      <origin xyz="-0.022 0 0"/>
+      <geometry><box size="0.04 0.04 0.03"/></geometry>
+    </collision>
   </link>
   <joint name="camera_joint" type="fixed">
@@ -208,5 +220,5 @@
     <child link="${lnk_cam}"/>
     <!-- Keep the camera body and optical origin ahead of the outer shell. -->
-    <origin xyz="${shell_length/2 + 0.03} 0 ${base_height + 0.05}" rpy="0 0 0"/>
+    <origin xyz="${shell_length/2 + 0.035} 0.075 0.185" rpy="0 0 0"/>
   </joint>
   <link name="${lnk_down_cam}">
@@ -217,15 +229,45 @@
     </inertial>
     <visual>
-      <geometry><box size="0.05 0.05 0.04"/></geometry>
-      <material name="down_camera_green"><color rgba="0.05 0.55 0.18 1.0"/></material>
-    </visual>
+      <origin xyz="-0.022 0 0"/>
+      <geometry><box size="0.04 0.04 0.03"/></geometry>
+      <material name="down_camera_green"><color rgba="0.04 0.06 0.09 1.0"/></material>
+    </visual>
+  <collision>
+      <origin xyz="-0.022 0 0"/>
+      <geometry><box size="0.04 0.04 0.03"/></geometry>
+    </collision>
   </link>
   <joint name="front_down_camera_joint" type="fixed">
     <parent link="${lnk_base}"/>
     <child link="${lnk_down_cam}"/>
-    <!-- Keep the lens ahead of the 0.42 m shell so the body is outside the image. -->
+    <!-- Separate the two lenses laterally; housings sit behind their optical origins. -->
     <!-- Positive pitch rotates the camera +X optical axis toward the floor. -->
-    <origin xyz="0.28 0 0.18" rpy="0 0.436332 0"/>
-  </joint>
+    <origin xyz="${shell_length/2 + 0.035} -0.075 0.185" rpy="0 0.436332 0"/>
+  </joint>
+  <!-- Low-friction support balls prevent the chassis rocking about its axle. -->
+  <xacro:macro name="support_ball" params="name x">
+    <link name="$(arg frame_prefix)${name}_link">
+      <inertial><mass value="0.05"/><inertia ixx="0.0000125" ixy="0" ixz="0" iyy="0.0000125" iyz="0" izz="0.0000125"/></inertial>
+      <visual><geometry><sphere radius="0.025"/></geometry><material name="black"/></visual>
+      <collision><geometry><sphere radius="0.025"/></geometry></collision>
+    </link>
+    <joint name="${name}_joint" type="fixed">
+      <parent link="${lnk_base}"/><child link="$(arg frame_prefix)${name}_link"/>
+      <origin xyz="${x} 0 0.025"/>
+    </joint>
+    <gazebo reference="$(arg frame_prefix)${name}_link">
+      <mu1>0.0</mu1><mu2>0.0</mu2><material>Gazebo/DarkGrey</material>
+    </gazebo>
+  </xacro:macro>
+  <xacro:support_ball name="front_support" x="0.165"/>
+  <xacro:support_ball name="rear_support" x="-0.165"/>
+  <!-- Explicit Gazebo materials survive URDF fixed-joint reduction. -->
+  <gazebo reference="${lnk_base}"><material>Gazebo/DarkGrey</material></gazebo>
+  <gazebo reference="$(arg frame_prefix)outer_shell_link"><material>Gazebo/White</material></gazebo>
+  <gazebo reference="${lnk_lw}"><material>Gazebo/Black</material></gazebo>
+  <gazebo reference="${lnk_rw}"><material>Gazebo/Black</material></gazebo>
+  <gazebo reference="${lnk_laser}"><material>Gazebo/Black</material></gazebo>
+  <gazebo reference="${lnk_cam}"><material>Gazebo/Black</material></gazebo>
+  <gazebo reference="${lnk_down_cam}"><material>Gazebo/Black</material></gazebo>
   <gazebo reference="${lnk_lw}">
     <mu1>2.0</mu1>
@@ -264,5 +306,4 @@
       <plugin name="ray_collision_filter" filename="$(arg collision_filter_plugin)">
         <own_category_bits>$(arg collision_bit)</own_category_bits>
-        <shell_link>$(arg frame_prefix)outer_shell_link</shell_link>
       </plugin>
       <plugin name="laser_controller" filename="libgazebo_ros_ray_sensor.so">
